File: bletest-2/power.kicad_sch (KiCad schematic)
At the start: 20 parts, among them J1 Conn_01x02, J4 Conn_01x02, J5 Conn_01x02, J6 Conn_01x02, U1 MAX40200AUK

Commit message: Full routing done
There are still a bunch of ERC violations.
Connections:
- net at C2.1, J1.1 (Pin_1), R1.1: now also U2.5 (VOUT)
- net at R1.2, R2.1: now also U2.4 (FB)
- no-connect marks 1 -> 8
Other:
- moved on the sheet: BT1, C1, C2, C3, C4, C5, D1, J1, J4, J5, J6, L1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

Commit message: Rev A of bletest
Finish cleanup, and remove last remaining violations.

There are a handful of silkscreen overlaps with explicit exclusions.
Parts:
- U2: value ~ -> TPS61070DDCR
- U3: value ~ -> MDBT53_1M
Other:
- company: (none) -> David Brown
- title: (none) -> BLETEXT-2
Changed lines of the file:
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@@
 	(generator "eeschema")
 	(generator_version "8.0")
-	(paper "A4")
+	(paper "A")
+	(title_block
+		(title "BLETEXT-2")
+		(date "2024-12-07")
+		(rev "REVA")
+		(company "David Brown")
+	)
 	(junction
 		(at 128.27 53.34)
@@
 			)
 		)
-		(property "Datasheet" "~"
+		(property "Datasheet" "https://www.digikey.com/en/products/detail/samsung-electro-mechanics/CL10A105KA8NNNC/3886760"
 			(at 114.3 124.46 0)
 			(effects
@@
 			)
 		)
-		(property "Datasheet" "~"
+		(property "Datasheet" "https://www.digikey.com/en/products/detail/taiyo-yuden/LBR2012T100K/1788937"
 			(at 92.71 120.65 0)
 			(effects
@@
 			)
 		)
-		(property "Datasheet" "https://datasheets.maximintegrated.com/en/ds/MAX40200.pdf"
+		(property "Datasheet" "https://www.digikey.com/en/products/detail/analog-devices-inc-maxim-integrated/MAX40200AUK-T/7392218"
 			(at 68.58 45.72 0)
 			(effects
@@
 			)
 		)
-		(property "Datasheet" "~"
+		(property "Datasheet" "https://www.digikey.com/en/products/detail/samsung-electro-mechanics/CL10A475KP8NNNC/3886702"
 			(at 49.53 114.3 0)
 			(effects
@@
 			)
 		)
-		(property "Datasheet" "~"
+		(property "Datasheet" "https://www.digikey.com/en/products/detail/samsung-electro-mechanics/CL10A105KA8NNNC/3886760"
 			(at 105.41 132.08 0)
 			(effects
@@
 			)
 		)
-		(property "Value" "~"
+		(property "Value" "MDBT53_1M"
 			(at 223.52 53.34 0)
 			(effects
@@
 			)
 		)
-		(property "Datasheet" ""
+		(property "Datasheet" "https://www.amazon.com/dp/B0B4BC8Z1V"
 			(at 223.52 76.2 0)
 			(effects
@@
 			)
 		)
-		(property "Datasheet" "~"
+		(property "Datasheet" "https://www.digikey.com/en/products/detail/te-connectivity-passive-product/CPF0603B1M0E/4966442"
 			(at 128.27 58.42 0)
 			(effects
@@
 			)
 		)
-		(property "Datasheet" "~"
+		(property "Datasheet" "https://www.amazon.com/gp/product/B0CGZQF3LR/"
 			(at 31.75 59.436 90)
 			(effects
@@
 			)
 		)
-		(property "Datasheet" "~"
+		(property "Datasheet" "https://www.digikey.com/en/products/detail/panasonic-electronic-components/ERA-3AEB184V/1465908"
 			(at 128.27 69.85 0)
 			(effects
@@
 			)
 		)
-		(property "Datasheet" "~"
+		(property "Datasheet" "https://www.digikey.com/en/products/detail/taiyo-yuden/CB2012T4R7M/1169459"
 			(at 92.71 53.34 0)
 			(effects
@@
 			)
 		)
-		(property "Datasheet" "~"
+		(property "Datasheet" "https://www.digikey.com/en/products/detail/micro-commercial-co/BAV19W-TP/717233"
 			(at 68.58 40.64 0)
 			(effects
@@
 			)
 		)
-		(property "Datasheet" "~"
+		(property "Datasheet" "https://www.digikey.com/en/products/detail/samsung-electro-mechanics/CL10A475KP8NNNC/3886702"
 			(at 142.24 59.69 0)
 			(effects
@@
 			)
 		)
-		(property "Datasheet" "~"
+		(property "Datasheet" "https://www.digikey.com/en/products/detail/panasonic-electronic-components/ERA-3AEB184V/1465908"
 			(at 204.47 66.04 0)
 			(effects
@@
 			)
 		)
-		(property "Datasheet" "~"
+		(property "Datasheet" "https://www.digikey.com/en/products/detail/taiyo-yuden/LBR2012T100K/1788937"
 			(at 92.71 128.27 0)
 			(effects
@@
 			)
 		)
-		(property "Value" "~"
+		(property "Value" "MDBT53_1M"
 			(at 58.42 127 0)
 			(effects
@@
 			)
 		)
-		(property "Datasheet" ""
+		(property "Datasheet" "https://www.amazon.com/dp/B0B4BC8Z1V"
 			(at 68.58 128.27 0)
 			(effects
@@
 			)
 		)
-		(property "Datasheet" "~"
+		(property "Datasheet" "https://www.digikey.com/en/products/detail/samsung-electro-mechanics/CL10A475KP8NNNC/3886702"
 			(at 88.9 63.5 0)
 			(effects
@@
 			)
 		)
-		(property "Value" "~"
+		(property "Value" "TPS61070DDCR"
 			(at 110.49 45.72 0)
 			(effects
@@
 			)
 		)
-		(property "Datasheet" ""
+		(property "Datasheet" "https://www.digikey.com/en/products/detail/texas-instruments/TPS61070DDCR/665929"
 			(at 107.95 60.96 0)
 			(effects
