File: bletest-2/switches.kicad_sch (KiCad schematic)
At the start: 8 parts, among them SW1 SW_Push, SW2 SW_Push, SW3 SW_Push, SW4 SW_Push

Commit message: Rev A of bletest
Finish cleanup, and remove last remaining violations.

There are a handful of silkscreen overlaps with explicit exclusions.
Other:
- company: (none) -> David Brown
- title: (none) -> BLETEXT-2
Changed lines of the file:
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@@
 	(generator "eeschema")
 	(generator_version "8.0")
-	(paper "A4")
+	(paper "A")
+	(title_block
+		(title "BLETEXT-2")
+		(date "2024-12-07")
+		(rev "REVA")
+		(company "David Brown")
+	)
 	(wire
 		(pts
@@
 			)
 		)
-		(property "Datasheet" "~"
+		(property "Datasheet" "https://www.digikey.com/en/products/detail/micro-commercial-co/BAV19W-TP/717233"
 			(at 134.62 71.12 0)
 			(effects
@@
 			)
 		)
-		(property "Datasheet" "~"
+		(property "Datasheet" "https://www.digikey.com/en/products/detail/micro-commercial-co/BAV19W-TP/717233"
 			(at 134.62 54.61 0)
 			(effects
@@
 			)
 		)
-		(property "Datasheet" "~"
+		(property "Datasheet" "https://www.digikey.com/en/products/detail/micro-commercial-co/BAV19W-TP/717233"
 			(at 72.39 71.12 0)
 			(effects
@@
 			)
 		)
-		(property "Datasheet" "~"
+		(property "Datasheet" "https://www.digikey.com/en/products/detail/micro-commercial-co/BAV19W-TP/717233"
 			(at 72.39 54.61 0)
 			(effects
