File: jolt2/jolt2-pim-left/power.kicad_sch (KiCad schematic)
At the start: 9 parts, among them J29 USB_C_Receptacle_USB2.0_14P, J30 Conn_ARM_JTAG_SWD_10

Commit message: jolt2-pim-left: Finalize routing
Parts:
- removed C1, C2: 10u, Capacitor_SMD:C_0603_1608Metric, symbol Device:C
- removed J29: USB_C_Receptacle_USB2.0_14P, davidb-keyboard-foot:USB_C_Receptacle_GCT_USB4085, symbol Connector:USB_C_Receptacle_USB2.0_14P
- removed U2: ~, davidb-keyboard-foot:AP2112M-SO8, symbol David Brown Keyboard Parts:AP2112M-3.3
- added J30: USB_C_Receptacle_USB2.0_14P, davidb-keyboard-foot:USB_C_Receptacle_GCT_USB4085, symbol Connector:USB_C_Receptacle_USB2.0_14P
- R3, R4: value R -> 5.1k
- renumbered J30 to J31
Connections:
- net +3.3V: no longer D1.4 (VDD), D2.4 (VDD)
- net GND: now also J30.A1 (GND), J30.A12 (GND), J30.B1 (GND), J30.B12 (GND), J30.S1 (SHIELD)
- net USB_D+: now also J30.A6 (D+), J30.B6 (D+)
- net USB_D-: now also J30.A7 (D-), J30.B7 (D-)
- net VBUS: now also D1.4 (VDD), D2.4 (VDD), J30.A4 (VBUS), J30.A9 (VBUS), J30.B4 (VBUS), J30.B9 (VBUS)
- net at R4.1: now also J30.A5 (CC1)
- net at R3.1: now also J30.B5 (CC2)
