File: jolt2/jolt2-tiny2040-left/jolt2-tiny2040-left.kicad_sch (KiCad schematic)
At the start: 5 parts

Commit message: jolt2-tiny204-left: Cleanup and route
Fix the designators for all of the pin headers.  This was mostly done
manually, naming them consistently for each component.

Perform manual routing.

This should be ready for REV A.
Parts:
- renumbered J to J29
Changed lines of the file:
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@@
 		(on_board yes)
 		(dnp no)
-		(property "Reference" "J"
+		(property "Reference" "J29"
 			(at 52.07 157.48 0)
 			(effects
@@
 			(project "jolt2-pim-left"
 				(path "/5e404b8e-7f18-4204-bb67-87c83d2db771"
-					(reference "J")
+					(reference "J29")
 					(unit 1)
 				)
