File: jolt2/jolt2-tiny2040-left/power.kicad_sch (KiCad schematic)
At the start: 1 part, among them J31 Conn_ARM_JTAG_SWD_10

Commit message: jolt2-tiny204-left: Cleanup and route
Fix the designators for all of the pin headers.  This was mostly done
manually, naming them consistently for each component.

Perform manual routing.

This should be ready for REV A.
Parts:
- renumbered J31 to J30
Changed lines of the file:
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@@
 		(dnp no)
 		(fields_autoplaced yes)
-		(property "Reference" "J31"
+		(property "Reference" "J30"
 			(at 144.78 118.1099 0)
 			(effects
@@
 			(project ""
 				(path "/5e404b8e-7f18-4204-bb67-87c83d2db771/a1c76de4-528d-42ab-822c-b4e73696ff22"
-					(reference "J31")
+					(reference "J30")
 					(unit 1)
 				)
