File: jolt2/jolt2-left/flash.kicad_sch (KiCad schematic)
At the start: 5 parts, among them SW1 SW_SPST, U3 W25Q128JVP

Commit message: jolt2: Prepare rev A
This is Rev A, being sent for production.
Parts:
- added J31: RJ45, Connector_RJ:RJ45_Amphenol_54602-x08_Horizontal, symbol Connector:RJ45
Connections:
- net GND: now also J31.2, J31.6, J31.7, J31.8
- new net SERRX: J31.1
- new net SERTX: J31.3
- new net VBUS: J31.4, J31.5

Commit message: jolt2-left: Add inter-board termination
Add 27 ohm resisters for termination on the inter-board protocol.
Parts:
- added R10, R9: 27, Resistor_SMD:R_0603_1608Metric_Pad0.98x0.95mm_HandSolder, symbol Device:R
Connections:
- net SERRX: now also R10.2; no longer J31.1
- net SERTX: now also R9.2; no longer J31.3
- new net: J31.3, R9.1
- new net: J31.1, R10.1
Other:
- note added: "Place R9, R10 near RP2040"
Changed lines of the file:
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@@
+	(wire
+		(pts
+			(xy 113.03 124.46) (xy 121.92 124.46)
+		)
+		(stroke
+			(width 0)
+			(type default)
+		)
+	)
 	(wire
 		(pts
@@
 	(wire
 		(pts
+			(xy 68.58 132.08) (xy 90.17 132.08)
+		)
+		(stroke
+			(width 0)
+			(type default)
+		)
+	)
+	(wire
+		(pts
 			(xy 68.58 129.54) (xy 74.93 129.54)
 		)
@@
 	(wire
 		(pts
+			(xy 90.17 134.62) (xy 105.41 134.62)
+		)
+		(stroke
+			(width 0)
+			(type default)
+		)
+	)
+	(wire
+		(pts
 			(xy 74.93 114.3) (xy 74.93 116.84)
 		)
@@
 	(wire
 		(pts
-			(xy 68.58 132.08) (xy 86.36 132.08)
+			(xy 90.17 132.08) (xy 90.17 134.62)
+		)
+		(stroke
+			(width 0)
+			(type default)
+		)
+	)
+	(wire
+		(pts
+			(xy 90.17 127) (xy 90.17 124.46)
 		)
 		(stroke
@@
 	(wire
 		(pts
-			(xy 68.58 127) (xy 86.36 127)
-		)
-		(stroke
-			(width 0)
-			(type default)
-		)
-	)
-	(wire
-		(pts
 			(xy 66.04 57.15) (xy 66.04 63.5)
 		)
@@
 	(wire
 		(pts
+			(xy 68.58 127) (xy 90.17 127)
+		)
+		(stroke
+			(width 0)
+			(type default)
+		)
+	)
+	(wire
+		(pts
 			(xy 66.04 63.5) (xy 73.66 63.5)
 		)
@@
 	(wire
 		(pts
+			(xy 90.17 124.46) (xy 105.41 124.46)
+		)
+		(stroke
+			(width 0)
+			(type default)
+		)
+	)
+	(wire
+		(pts
 			(xy 62.23 53.34) (xy 62.23 57.15)
 		)
@@
 	(wire
 		(pts
+			(xy 113.03 134.62) (xy 121.92 134.62)
+		)
+		(stroke
+			(width 0)
+			(type default)
+		)
+	)
+	(wire
+		(pts
 			(xy 58.42 63.5) (xy 66.04 63.5)
 		)
@@
 			(width 0)
 			(type default)
+		)
+	)
+	(text "Place R9, R10 near RP2040"
+		(exclude_from_sim no)
+		(at 135.382 115.824 0)
+		(effects
+			(font
+				(size 1.27 1.27)
+			)
 		)
 	)
@@
 	(global_label "SERRX"
 		(shape input)
-		(at 86.36 132.08 0)
+		(at 121.92 134.62 0)
 		(fields_autoplaced yes)
 		(effects
@@
 		)
 		(property "Intersheetrefs" "${INTERSHEET_REFS}"
-			(at 95.4532 132.08 0)
+			(at 131.0132 134.62 0)
 			(effects
 				(font
@@
 	(global_label "SERTX"
 		(shape input)
-		(at 86.36 127 0)
+		(at 121.92 124.46 0)
 		(fields_autoplaced yes)
 		(effects
@@
 		)
 		(property "Intersheetrefs" "${INTERSHEET_REFS}"
-			(at 95.1508 127 0)
+			(at 130.7108 124.46 0)
 			(effects
 				(font
@@
 	)
 	(symbol
+		(lib_id "Device:R")
+		(at 109.22 124.46 90)
+		(unit 1)
+		(exclude_from_sim no)
+		(in_bom yes)
+		(on_board yes)
+		(dnp no)
+		(fields_autoplaced yes)
+		(property "Reference" "R9"
+			(at 109.22 118.11 90)
+			(effects
+				(font
+					(size 1.27 1.27)
+				)
+			)
+		)
+		(property "Value" "27"
+			(at 109.22 120.65 90)
+			(effects
+				(font
+					(size 1.27 1.27)
+				)
+			)
+		)
+		(property "Footprint" "Resistor_SMD:R_0603_1608Metric_Pad0.98x0.95mm_HandSolder"
+			(at 109.22 126.238 90)
+			(effects
+				(font
+					(size 1.27 1.27)
+				)
+				(hide yes)
+			)
+		)
+		(property "Datasheet" "~"
+			(at 109.22 124.46 0)
+			(effects
+				(font
+					(size 1.27 1.27)
+				)
+				(hide yes)
+			)
+		)
+		(property "Description" "Resistor"
+			(at 109.22 124.46 0)
+			(effects
+				(font
+					(size 1.27 1.27)
+				)
+				(hide yes)
+			)
+		)
+		(pin "2"
+		)
+		(pin "1"
+		)
+		(instances
+			(project ""
+				(path "/5e404b8e-7f18-4204-bb67-87c83d2db771/83902f8d-393e-44e1-a57d-86e4f1895520"
+					(reference "R9")
+					(unit 1)
+				)
+			)
+		)
+	)
+	(symbol
 		(lib_id "power:VBUS")
 		(at 82.55 107.95 0)
@@
 					(unit 1)
 				)
+			)
+		)
+	)
+	(symbol
+		(lib_id "Device:R")
+		(at 109.22 134.62 90)
+		(unit 1)
+		(exclude_from_sim no)
+		(in_bom yes)
+		(on_board yes)
+		(dnp no)
+		(property "Reference" "R10"
+			(at 109.474 137.414 90)
+			(effects
+				(font
+					(size 1.27 1.27)
+				)
+			)
+		)
+		(property "Value" "27"
+			(at 109.22 131.318 90)
+			(effects
+				(font
+					(size 1.27 1.27)
+				)
+			)
+		)
+		(property "Footprint" "Resistor_SMD:R_0603_1608Metric_Pad0.98x0.95mm_HandSolder"
+			(at 109.22 136.398 90)
+			(effects
+				(font
+					(size 1.27 1.27)
+				)
+				(hide yes)
+			)
+		)
+		(property "Datasheet" "~"
+			(at 109.22 134.62 0)
+			(effects
+				(font
+					(size 1.27 1.27)
+				)
+				(hide yes)
+			)
+		)
+		(property "Description" "Resistor"
+			(at 109.22 134.62 0)
+			(effects
+				(font
+					(size 1.27 1.27)
+				)
+				(hide yes)
+			)
+		)
+		(pin "2"
+		)
+		(pin "1"
+		)
+		(instances
+			(project ""
+				(path "/5e404b8e-7f18-4204-bb67-87c83d2db771/83902f8d-393e-44e1-a57d-86e4f1895520"
+					(reference "R10")
+					(unit 1)
+				)

Commit message: Various PCB updates
This is before fixing the footprint for the WS2812. Turns out there is a
ws2812 MINI, and a MINI-HS, and they have very different footprints.
Parts:
- C16: value C -> 100n
Changed lines of the file:
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@@
 			)
 		)
-		(property "Value" "C"
+		(property "Value" "100n"
 			(at 102.87 53.3399 0)
 			(effects
