File: jolt3/jolt3-right/jolt3-right.kicad_pcb (KiCad board)
At the start: 2 copper layers, 151 x 98 mm, 33 parts, among them J1 Conn_01x02_Pin, J10 Conn_01x02_Pin, J11 Conn_01x02_Pin, J12 Conn_01x02_Pin, J13 Conn_01x02_Pin, J14 Conn_01x02_Pin, J15 Conn_01x02_Pin, J16 Conn_01x02_Pin, J17 Conn_01x02_Pin, J18 Conn_01x02_Pin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

Commit message: Jolt 3: Rev A for 3 boards
Send Rev A out for jolt3-left, jolt3-right, and j3-mez-2040.
Parts:
- moved R1 139.1 mm to (25.8, 132.9)
- moved R2 139.1 mm to (25.8, 135.4)
- moved BT1 94.0 mm to (56.0, 93.5), turned to 0 degrees
- moved J25 73.1 mm to (93.0, 138.3), turned to 10 degrees
- moved J28 72.6 mm to (36.8, 148.2), turned to 10 degrees
- moved J26 69.0 mm to (95.0, 150.2), turned to -170 degrees
- moved J27 68.5 mm to (38.9, 160.1), turned to -170 degrees
- moved J31 29.6 mm to (28.2, 126.5)
- moved J29 14.5 mm to (34.6, 133.5), turned to 90 degrees
Connections:
- J31 pad 1: /SER-RX -> /SER-TX
- J31 pad 3: /SER-TX -> /SER-RX
Routing:
- net /ROW-A: track 0.00 -> 242.0 mm, vias 0 -> 1
- net /ROW-B: track 0.00 -> 206.5 mm, vias 0 -> 1
- net /ROW-C: track 0.00 -> 194.2 mm, vias 0 -> 2
- net /ROW-D: track 0.00 -> 154.5 mm, vias 0 -> 1
- net /COL-A: track 0.00 -> 141.1 mm, vias 0 -> 1
- net /ROW-E: track 0.00 -> 124.0 mm
- net /ROW-F: track 0.00 -> 113.2 mm
- net /COL-B: track 0.00 -> 112.2 mm, vias 0 -> 1
- net /COL-C: track 0.00 -> 88.6 mm, vias 0 -> 2
- net /COL-D: track 0.00 -> 64.0 mm
- net GND: track 0.00 -> 58.4 mm
- net /SDA: track 0.00 -> 29.9 mm
- net Net-(BT1-+): track 0.00 -> 29.1 mm, vias 0 -> 1
- net /SCL: track 0.00 -> 24.2 mm
- net VBUS: track 0.00 -> 20.0 mm
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Other:
- board text added: "Jolt 3 - Right REV A"
- board text removed: "Jolt 2 - Left REV B"

Commit message: Update for latest KiCad
This seems to have done a rewrite of uuids within the files.
Parts:
- moved BT1 10.1 mm to (66.1, 93.0)
- moved J31 4.08 mm to (28.2, 122.5)
Routing:
- net /ROW-C: track 194.2 -> 157.9 mm, vias 2 -> 3
- net GND: track 58.4 -> 68.4 mm, vias 0 -> 1
- net Net-(BT1-+): track 29.1 -> 38.8 mm
- net /SDA: track 29.9 -> 34.0 mm
- net /SER-RX: track 12.5 -> 16.6 mm
- net /SCL: track 24.2 -> 28.2 mm
- net /SER-TX: track 11.8 -> 15.7 mm
- net VBUS: track 20.0 -> 22.2 mm, vias 0 -> 1
Other:
- board text added: "Jolt 3 - Right REV B"
- board text removed: "Jolt 3 - Right REV A"
