File: mesa1/mesa1-left/mesa1-left.kicad_pcb (KiCad board)
At the start: 2 copper layers, 133 x 94 mm, 38 parts, among them J1 RJ45, J2 Tag-Connect TC2030

Commit message: Update the mesa1 for Rev A
This version rejects compatibility with older designs, in order to make
routing a lot easier.
Connections:
- net /ROW_6 renamed /COL_6
- A1 pad 0: /ROW_1 -> /ROW_E
- A1 pad 1: /ROW_2 -> /ROW_D
- A1 pad 2: /ROW_3 -> /ROW_C
- A1 pad 3: /ROW_4 -> /ROW_B
- A1 pad 4: /ROW_5 -> /ROW_A
- A1 pad 6: /COL_A -> /COL_5
- A1 pad 7: /COL_B -> /COL_4
- A1 pad A0: /COL_C -> /RGB
- A1 pad A1: /COL_D -> /COL_1
- A1 pad A2: /COL_E -> /COL_2
- A1 pad A3: /RGB -> /COL_3
- D_LA0 pad 1: /ROW_2 -> /ROW_E
- D_LF1 pad 1: /ROW_1 -> /ROW_A
- D_LF2 pad 1: /ROW_2 -> /ROW_C
- D_LH0 pad 1: /ROW_3 -> /ROW_B
- D_LK0 pad 1: /ROW_3 -> /ROW_C
- D_LNUM0 pad 1: /ROW_1 -> /ROW_E
- D_LO0 pad 1: /ROW_3 -> /ROW_E
- D_LP0 pad 1: /ROW_1 -> /ROW_B
- D_LR0 pad 1: /ROW_1 -> /ROW_D
- D_LS0 pad 1: /ROW_1 -> /ROW_C
- D_LS1 pad 1: /ROW_2 -> /ROW_B
- D_LS2 pad 1: /ROW_3 -> /ROW_D
- D_LSTAR0 pad 1: /ROW_3 -> /ROW_A
- D_LT0 pad 1: /ROW_2 -> /ROW_A
- D_LW0 pad 1: /ROW_2 -> /ROW_D
- J1 pad 1: /ROW_4 -> /COL_4
- J1 pad 2: /ROW_5 -> /COL_5
- J1 pad 4: /COL_A -> /ROW_A
- J1 pad 5: /COL_B -> /ROW_B
- J1 pad 6: /COL_C -> /ROW_C
- J1 pad 7: /COL_D -> /ROW_D
- J1 pad 8: /COL_E -> /ROW_E
- L-A0 pad 1: /COL_E -> /COL_2
- L-H0 pad 1: /COL_C -> /COL_2
- L-K0 pad 1: /COL_B -> /COL_3
- L-O0 pad 1: /COL_E -> /COL_3
- L-P0 pad 1: /COL_C -> /COL_1
- L-R0 pad 1: /COL_D -> /COL_2
- L-S0 pad 1: /COL_B -> /COL_2
- L-STAR0 pad 1: /COL_A -> /COL_2
- L-T0 pad 1: /COL_B -> /COL_3
- L-W0 pad 1: /COL_C -> /COL_1
- LF1 pad 1: /COL_A -> /COL_1
- LF2 pad 1: /COL_A -> /COL_1
- LNUM0 pad 1: /COL_E -> /COL_1
- LS1 pad 1: /COL_D -> /COL_3
- LS2 pad 1: /COL_D -> /COL_3
Routing:
- net /COL_2: track 0.00 -> 219.7 mm, vias 0 -> 4
- net /COL_1: track 0.00 -> 215.6 mm, vias 0 -> 1
- net /ROW_C: track 0.00 -> 187.3 mm, vias 0 -> 1
- net /COL_3: track 0.00 -> 185.7 mm, vias 0 -> 3
- net /ROW_A: track 0.00 -> 181.4 mm, vias 0 -> 2
- net /ROW_B: track 0.00 -> 133.7 mm, vias 0 -> 1
- net /ROW_D: track 0.00 -> 128.8 mm
- net /ROW_E: track 0.00 -> 124.7 mm, vias 0 -> 2
- net /GND: track 0.00 -> 114.1 mm, vias 0 -> 4
- net /+5V: track 0.00 -> 79.4 mm, vias 0 -> 2
- net /+3V3: track 0.00 -> 46.9 mm, vias 0 -> 2
- net /RGB: track 0.00 -> 46.4 mm, vias 0 -> 2
- net /COL_6: track 0.00 -> 39.2 mm
- net /COL_5: track 0.00 -> 37.3 mm
- net /COL_4: track 0.00 -> 29.5 mm
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Other:
- board text added: "Mesa1-left Rev A tangybbq/keyboards"
