File: mesa1/mesa1-left/mesa1-left.kicad_sch (KiCad schematic)
At the start: 38 parts, among them J1 RJ45, J2 Tag-Connect TC2030

Commit message: Update the mesa1 for Rev A
This version rejects compatibility with older designs, in order to make
routing a lot easier.
Connections:
- net RGB: now also A1.A0 (A0/GP26); no longer A1.A3 (A3/GP29)
- removed net COL_A: A1.6 (GP6), J1.4, L-STAR0.1 (A), LF1.1 (A), LF2.1 (A)
- removed net COL_B: A1.7 (GP7), J1.5, L-K0.1 (A), L-S0.1 (A), L-T0.1 (A)
- removed net COL_C: A1.A0 (A0/GP26), J1.6, L-H0.1 (A), L-P0.1 (A), L-W0.1 (A)
- removed net COL_D: A1.A1 (A1/GP27), J1.7, L-R0.1 (A), LS1.1 (A), LS2.1 (A)
- removed net COL_E: A1.A2 (A2/GP28), J1.8, L-A0.1 (A), L-O0.1 (A), LNUM0.1 (A)
- removed net ROW_1: A1.0 (GP0), D_LF1.1 (K), D_LNUM0.1 (K), D_LP0.1 (K), D_LR0.1 (K), D_LS0.1 (K)
- removed net ROW_2: A1.1 (GP1), D_LA0.1 (K), D_LF2.1 (K), D_LS1.1 (K), D_LT0.1 (K), D_LW0.1 (K)
- removed net ROW_3: A1.2 (GP2), D_LH0.1 (K), D_LK0.1 (K), D_LO0.1 (K), D_LS2.1 (K), D_LSTAR0.1 (K)
- net ROW_4 renamed COL_4
- net COL_4: now also A1.7 (GP7); no longer A1.3 (GP3)
- net ROW_5 renamed COL_5
- net COL_5: now also A1.6 (GP6); no longer A1.4 (GP4)
- net ROW_6 renamed COL_6
- new net COL_1: A1.A1 (A1/GP27), L-P0.1 (A), L-W0.1 (A), LF1.1 (A), LF2.1 (A), LNUM0.1 (A)
- new net COL_2: A1.A2 (A2/GP28), L-A0.1 (A), L-H0.1 (A), L-R0.1 (A), L-S0.1 (A), L-STAR0.1 (A)
- new net COL_3: A1.A3 (A3/GP29), L-K0.1 (A), L-O0.1 (A), L-T0.1 (A), LS1.1 (A), LS2.1 (A)
- new net ROW_A: A1.4 (GP4), D_LF1.1 (K), D_LSTAR0.1 (K), D_LT0.1 (K), J1.4
- new net ROW_B: A1.3 (GP3), D_LH0.1 (K), D_LP0.1 (K), D_LS1.1 (K), J1.5
- new net ROW_C: A1.2 (GP2), D_LF2.1 (K), D_LK0.1 (K), D_LS0.1 (K), J1.6
- new net ROW_D: A1.1 (GP1), D_LR0.1 (K), D_LS2.1 (K), D_LW0.1 (K), J1.7
- new net ROW_E: A1.0 (GP0), D_LA0.1 (K), D_LNUM0.1 (K), D_LO0.1 (K), J1.8
Other:
- title: (none) -> mesa1-left
- moved on the sheet: LED1, LED2, LED3, LED4
