File: mesa1/mesa1-right/mesa1-right.kicad_pcb (KiCad board)
At the start: 2 copper layers, 133 x 94 mm, 31 parts, among them J1 RJ45

Commit message: Update the mesa1 for Rev A
This version rejects compatibility with older designs, in order to make
routing a lot easier.
Connections:
- D_RB0 pad 1: /ROW_5 -> /ROW_D
- D_RD0 pad 1: /ROW_4 -> /ROW_A
- D_RE0 pad 1: /ROW_6 -> /ROW_E
- D_RF0 pad 1: /ROW_6 -> /ROW_B
- D_RG0 pad 1: /ROW_6 -> /ROW_C
- D_RL0 pad 1: /ROW_5 -> /ROW_A
- D_RNUM0 pad 1: /ROW_4 -> /ROW_E
- D_RP0 pad 1: /ROW_4 -> /ROW_B
- D_RR0 pad 1: /ROW_4 -> /ROW_D
- D_RS3 pad 1: /ROW_5 -> /ROW_B
- D_RS4 pad 1: /ROW_6 -> /ROW_D
- D_RT0 pad 1: /ROW_6 -> /ROW_A
- D_RU0 pad 1: /ROW_5 -> /ROW_E
- D_RZ0 pad 1: /ROW_5 -> /ROW_C
- D_TS0 pad 1: /ROW_4 -> /ROW_C
- J1 pad 1: /ROW_4 -> /COL_4
- J1 pad 2: /ROW_5 -> /COL_5
- J1 pad 3: /ROW_6 -> /COL_6
- J1 pad 4: /COL_A -> /ROW_A
- J1 pad 5: /COL_B -> /ROW_B
- J1 pad 6: /COL_C -> /ROW_C
- J1 pad 7: /COL_D -> /ROW_D
- J1 pad 8: /COL_E -> /ROW_E
- RB0 pad 1: /COL_C -> /COL_4
- RD0 pad 1: /COL_A -> /COL_4
- RE0 pad 1: /COL_E -> /COL_6
- RF0 pad 1: /COL_C -> /COL_5
- RG0 pad 1: /COL_B -> /COL_6
- RL0 pad 1: /COL_B -> /COL_6
- RNUM0 pad 1: /COL_E -> /COL_4
- RP0 pad 1: /COL_C -> /COL_4
- RR0 pad 1: /COL_D -> /COL_5
- RS3 pad 1: /COL_D -> /COL_6
- RS4 pad 1: /COL_D -> /COL_6
- RT0 pad 1: /COL_A -> /COL_5
- RU0 pad 1: /COL_E -> /COL_5
- RZ0 pad 1: /COL_A -> /COL_4
- TS0 pad 1: /COL_B -> /COL_5
Routing:
- net /COL_4: track 0.00 -> 180.0 mm, vias 0 -> 2
- net /COL_6: track 0.00 -> 149.1 mm
- net /COL_5: track 0.00 -> 146.4 mm
- net /ROW_C: track 0.00 -> 141.3 mm, vias 0 -> 3
- net /ROW_A: track 0.00 -> 137.4 mm, vias 0 -> 1
- net /ROW_B: track 0.00 -> 96.4 mm, vias 0 -> 1
- net /ROW_D: track 0.00 -> 89.7 mm, vias 0 -> 2
- net /ROW_E: track 0.00 -> 86.6 mm
- net Net-(D_TS0-A): track 0.00 -> 11.7 mm
- net Net-(D_RP0-A): track 0.00 -> 11.7 mm
- net Net-(D_RG0-A): track 0.00 -> 11.7 mm
- net Net-(D_RF0-A): track 0.00 -> 11.7 mm
- net Net-(D_RD0-A): track 0.00 -> 11.7 mm
- net Net-(D_RB0-A): track 0.00 -> 11.7 mm
- net Net-(D_RL0-A): track 0.00 -> 11.7 mm
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Other:
- board text added: "Mesa1-left Rev A tangybbq/keyboards"
