File: mesa1/mesa1-right/mesa1-right.kicad_sch (KiCad schematic)
At the start: 31 parts, among them J1 RJ45

Commit message: Update the mesa1 for Rev A
This version rejects compatibility with older designs, in order to make
routing a lot easier.
Connections:
- net COL_A renamed COL_4
- net COL_4: now also J1.1, RB0.1 (A), RNUM0.1 (A), RP0.1 (A); no longer J1.4, RT0.1 (A)
- net COL_B renamed COL_6
- net COL_6: now also J1.3, RE0.1 (A), RS3.1 (A), RS4.1 (A); no longer J1.5, TS0.1 (A)
- removed net COL_C: J1.6, RB0.1 (A), RF0.1 (A), RP0.1 (A)
- removed net COL_D: J1.7, RR0.1 (A), RS3.1 (A), RS4.1 (A)
- removed net COL_E: J1.8, RE0.1 (A), RNUM0.1 (A), RU0.1 (A)
- removed net ROW_4: D_RD0.1 (K), D_RNUM0.1 (K), D_RP0.1 (K), D_RR0.1 (K), D_TS0.1 (K), J1.1
- removed net ROW_5: D_RB0.1 (K), D_RL0.1 (K), D_RS3.1 (K), D_RU0.1 (K), D_RZ0.1 (K), J1.2
- removed net ROW_6: D_RE0.1 (K), D_RF0.1 (K), D_RG0.1 (K), D_RS4.1 (K), D_RT0.1 (K), J1.3
- new net COL_5: J1.2, RF0.1 (A), RR0.1 (A), RT0.1 (A), RU0.1 (A), TS0.1 (A)
- new net ROW_A: D_RD0.1 (K), D_RL0.1 (K), D_RT0.1 (K), J1.4
- new net ROW_B: D_RF0.1 (K), D_RP0.1 (K), D_RS3.1 (K), J1.5
- new net ROW_C: D_RG0.1 (K), D_RZ0.1 (K), D_TS0.1 (K), J1.6
- new net ROW_D: D_RB0.1 (K), D_RR0.1 (K), D_RS4.1 (K), J1.7
- new net ROW_E: D_RE0.1 (K), D_RNUM0.1 (K), D_RU0.1 (K), J1.8
Other:
- title: (none) -> mesa1-right
- moved on the sheet: D_RE0, D_RNUM0, D_RR0, D_RS3, D_RS4, D_RU0, RE0, RNUM0, RR0, RS3, RS4, RU0
