File: mesa2/mesa2/mesa2.kicad_sch (KiCad schematic)
At the start: 53 parts, among them J2 Tag-Connect TC2030

Commit message: Do the Rev B schematic work for mesa2
Delete the outer pinky keys and repair the column pairing, the two
changes that live entirely in the schematic. SW_LR1, SW_RR1 and their
diodes are gone along with the eight wire stubs that tied those grid
cells to their row and column buses, leaving 18 keys in the 5x4 grid.

The columns now pair by finger rather than mirroring the two hands, so
COL_1 is the pinky on both sides instead of the left pinky and the right
index. Done by moving the right-hand symbols between grid cells, which
leaves every wire where it was. ERC shows no new violations.

Add revb.py, which reads Rev A's key positions straight out of the board
and applies the geometry changes: the pinky caps rotate 90 degrees and
the SP thumb keys move 1 mm closer to BK, landing on the 17 mm pitch the
finger rows use. The earlier placement.json and sw.json snapshots predate
the 5 degree hand rotation and no longer match the PCB, so the board is
what revb.py reads. The PCB itself is untouched: applying the new
placement needs a running KiCad.

Assisted-by: Claude:opus-5
Parts:
- removed D_LR1, D_RR1: 1N4148W, Diode_SMD:D_SOD-123, symbol Device:D
- removed SW_LR1, SW_RR1: SW_PG1350, mesa1:Kailh_socket_PG1350, symbol Switch:SW_SPST
Connections:
- net COL_1: now also D_RA1.1 (K); no longer D_RE1.1 (K), D_RI1.1 (K)
- net COL_2: now also D_RO1.1 (K), D_RS1.1 (K); no longer D_RN1.1 (K), D_RT1.1 (K)
- net COL_3: now also D_RN1.1 (K), D_RT1.1 (K); no longer D_RO1.1 (K), D_RS1.1 (K)
- net COL_4: now also D_RE1.1 (K), D_RI1.1 (K); no longer D_RA1.1 (K)
Other:
- moved on the sheet: D_RA1, D_RE1, D_RI1, D_RN1, D_RO1, D_RS1, D_RT1, SW_RA1, SW_RE1, SW_RI1, SW_RN1, SW_RO1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
