File: jolt3/j3-mez-2040/j3-mez-2040.kicad_pcb (KiCad board)
At the start: 4 copper layers, 38 x 38 mm, 37 parts, among them J2 Conn_ARM_SWD_TagConnect_TC2030, J29 USB_C_Receptacle_USB2.0_14P, SW1 SW_SPST, SW2 SW_SPST, U1 RP2040, U2 AP2112-M3.3, U3 W25Q128JVP, Y1 ABM8-272-T3

Commit message: Move j3-mez-2040 to KiCad 10 and reseat U3 as SOIC-8
Opening the board in KiCad 10 rewrites it wholesale: the copper and user
layers are renumbered, vias gain the tenting/covering/plugging/capping
attributes, the numeric net table is replaced by net names quoted at each
pad, the duplicated Footprint properties are dropped, and -90 degree
rotations normalise to 270.  None of that is a design change; all 427
track segments survive untouched.

Riding along is the first item from TASKS.md: U3, the QSPI flash, swaps
from WSON-8 to Package_SO:SOIC-8_5.3x5.3mm_P1.27mm so JLC can assemble it,
which cost one via in the re-route.  The two changes cannot be separated
because the format migration rewrote every line of the file.

Note that flash.kicad_sch still gives U3 the WSON-8 footprint, so the next
update-PCB-from-schematic would undo this.  The schematic side of the swap,
and the SW1/SW2 tactile swap, remain open in TASKS.md.
Parts:
- U3: footprint Package_SON:WSON-8-1EP_6x5mm_P1.27mm_EP3.4x4.3mm -> Package_SO:SOIC-8_5.3x5.3mm_P1.27mm
