File: mesa3/mesa3-left/mesa3-left.kicad_sch (KiCad schematic)
At the start: 55 parts, among them J2 Tag-Connect TC2030

Commit message: Split the Mesa 3 into left and right halves
Each half now carries its own nine keys, its own outline and its own
routing. The left keeps the Tiny2040, the LEDs, the Tag-Connect and the
reset pad; the right is switches, diodes and the RJ-45 and nothing else,
with no power and no ground anywhere on it.

The two checks that mattered both hold. The RJ-45 pinout is identical at
both ends, so a straight-through cable is correct -- the pin order runs
opposite between the halves, which is what a part that cannot be mirrored
does, and does not matter since the nets match. And all eighteen keys
keep their exact mesa2 column and row, so one keymap still serves Rev B
and both halves.

Record the review findings as accepted rather than outstanding, and
correct LAYOUT.md: the unconnected GND that DRC reports is a false
positive. The symbol ties the module's ground pads into one net, so DRC
wants copper between them, but the module commons them internally and
the board does not need to.

Assisted-by: Claude:opus-5
Parts:
- removed D_RA1, D_RBK1, D_RE1, D_RI1, D_RN1, D_RO1, D_RS1, D_RSP1, D_RT1: 1N4148W, Diode_SMD:D_SOD-123, symbol Device:D
- removed H4, H6: MountingHole, MountingHole:MountingHole_2.2mm_M2, symbol Mechanical:MountingHole
- removed SW_RA1, SW_RBK1, SW_RE1, SW_RI1, SW_RN1, SW_RO1, SW_RS1, SW_RSP1, SW_RT1: SW_PG1350, mesa1:Kailh_socket_PG1350, symbol Switch:SW_SPST
- added J1: RJ45, Connector_RJ:RJ45_Amphenol_54602-x08_Horizontal, symbol Connector:RJ45
Connections:
- net COL_1: now also J1.2
- net COL_2: now also J1.3
- net COL_3: now also J1.4
- net COL_4: now also J1.5
- net COL_5: now also J1.8
- net ROW_C: now also J1.7
- net ROW_D: now also J1.6

Commit message: Add the FN mode key to mesa3-left and place it
The Rev B change lands on the left half: SW_LFN1 and D_LFN1, one key
inboard of the near-row index key, for mode switching.  It takes the slot
the dropped outer pinky left free — SW_LFN1 pad 1 on ROW_A, D_LFN1 pad 1
on COL_1 — so it costs no GPIO, and since pinky A sits on ROW_B the two
share COL_1 without colliding.

Placement comes from fnkey.py rather than the mouse.  The key was first
dropped by hand at (112.700, 84.700), which measured 17.053 mm along
SW_LE1's local X with 0.435 mm of lateral drift; the computed position is
(113.272, 85.571) at a clean local (18, 0), a move of 1.042 mm.  D_LFN1
follows at the usual (0, -4.876) offset.  The cap gap against SW_LE1 comes
out at 0.500 mm exactly, which is the board's new worst gap, just inside
the 0.496 mm the thumb pair already had.  LAYOUT.md records both positions
and the rule that produced them.

Two things this commit deliberately contains.  All routing is gone — 308
segments and 41 vias — removed on purpose, to be redone once the non-switch
components settle; the four zones are untouched.  And the support parts
have moved to clear the new key: the four LEDs and their caps, D1, JP1, J2
and the reset pad.  Those are hand-placed and not governed by LAYOUT.md,
which speaks for the keys.

Watch JP1: it clears the new keycap edge by 0.52 mm.  Nothing sits under
the cap or the switch body, but JP1 is the bypass jumper across D1 and an
iron has to reach it.
Parts:
- added D_LFN1: 1N4148W, Diode_SMD:D_SOD-123, symbol Device:D
- added SW_LFN1: SW_PG1350, mesa1:Kailh_socket_PG1350, symbol Switch:SW_SPST
Connections:
- net COL_1: now also D_LFN1.1 (K)
- net ROW_A: now also SW_LFN1.1 (A)
- new net: D_LFN1.2 (A), SW_LFN1.2 (B)
Changed lines of the file:
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@@
+	(wire
+		(pts
+			(xy 27.94 34.29) (xy 22.86 34.29)
+		)
+		(stroke
+			(width 0)
+			(type default)
+		)
+	)
 	(wire
 		(pts
@@
 	(wire
 		(pts
+			(xy 22.86 34.29) (xy 22.86 22.86)
+		)
+		(stroke
+			(width 0)
+			(type default)
+		)
+	)
+	(wire
+		(pts
 			(xy 102.87 99.06) (xy 105.41 99.06)
 		)
@@
 		(pts
 			(xy 88.9 165.1) (xy 101.6 165.1)
+		)
+		(stroke
+			(width 0)
+			(type default)
+		)
+	)
+	(wire
+		(pts
+			(xy 38.1 34.29) (xy 46.99 34.29)
 		)
 		(stroke
@@
 				(path "/6762c7a5-6197-445d-9eb4-2a300e3d331b"
 					(reference "SW_LE1")
+					(unit 1)
+				)
+			)
+		)
+	)
+	(symbol
+		(lib_id "Device:D")
+		(at 50.8 34.29 180)
+		(unit 1)
+		(body_style 1)
+		(exclude_from_sim no)
+		(in_bom yes)
+		(on_board yes)
+		(in_pos_files yes)
+		(dnp no)
+		(property "Reference" "D_LFN1"
+			(at 50.8 30.48 0)
+			(show_name no)
+			(do_not_autoplace no)
+			(effects
+				(font
+					(size 1.27 1.27)
+				)
+			)
+		)
+		(property "Value" "1N4148W"
+			(at 50.8 38.1 0)
+			(show_name no)
+			(do_not_autoplace no)
+			(effects
+				(font
+					(size 1.27 1.27)
+				)
+			)
+		)
+		(property "Footprint" "Diode_SMD:D_SOD-123"
+			(at 50.8 34.29 0)
+			(hide yes)
+			(show_name no)
+			(do_not_autoplace no)
+			(effects
+				(font
+					(size 1.27 1.27)
+				)
+			)
+		)
+		(property "Datasheet" ""
+			(at 50.8 34.29 0)
+			(hide yes)
+			(show_name no)
+			(do_not_autoplace no)
+			(effects
+				(font
+					(size 1.27 1.27)
+				)
+			)
+		)
+		(property "Description" ""
+			(at 50.8 34.29 0)
+			(show_name no)
+			(do_not_autoplace no)
+			(effects
+				(font
+					(size 1.27 1.27)
+				)
+			)
+		)
+		(pin "2"
+		)
+		(pin "1"
+		)
+		(instances
+			(project "mesa3-left"
+				(path "/6762c7a5-6197-445d-9eb4-2a300e3d331b"
+					(reference "D_LFN1")
 					(unit 1)
 				)
@@
 					(unit 1)
 				)
+			)
+		)
+	)
+	(symbol
+		(lib_id "Switch:SW_SPST")
+		(at 33.02 34.29 0)
+		(unit 1)
+		(body_style 1)
+		(exclude_from_sim no)
+		(in_bom yes)
+		(on_board yes)
+		(in_pos_files yes)
+		(dnp no)
+		(property "Reference" "SW_LFN1"
+			(at 33.02 30.48 0)
+			(show_name no)
+			(do_not_autoplace no)
+			(effects
+				(font
+					(size 1.27 1.27)
+				)
+			)
+		)
+		(property "Value" "SW_PG1350"
+			(at 33.02 38.1 0)
+			(show_name no)
+			(do_not_autoplace no)
+			(effects
+				(font
+					(size 1.27 1.27)
+				)
+			)
+		)
+		(property "Footprint" "mesa1:Kailh_socket_PG1350"
+			(at 33.02 34.29 0)
+			(hide yes)
+			(show_name no)
+			(do_not_autoplace no)
+			(effects
+				(font
+					(size 1.27 1.27)
+				)
+			)
+		)
+		(property "Datasheet" ""
+			(at 33.02 34.29 0)
+			(hide yes)
+			(show_name no)
+			(do_not_autoplace no)
+			(effects
+				(font
+					(size 1.27 1.27)
+				)
+			)
+		)
+		(property "Description" ""
+			(at 33.02 34.29 0)
+			(show_name no)
+			(do_not_autoplace no)
+			(effects
+				(font
+					(size 1.27 1.27)
+				)
+			)
+		)
+		(pin "1"
+		)
+		(pin "2"
+		)
+		(instances
+			(project "mesa3-left"
+				(path "/6762c7a5-6197-445d-9eb4-2a300e3d331b"
+					(reference "SW_LFN1")
+					(unit 1)
+				)
