File: mesa3/mesa3-right/mesa3-right.kicad_sch (KiCad schematic)
At the start: 55 parts, among them J2 Tag-Connect TC2030

Commit message: Split the Mesa 3 into left and right halves
Each half now carries its own nine keys, its own outline and its own
routing. The left keeps the Tiny2040, the LEDs, the Tag-Connect and the
reset pad; the right is switches, diodes and the RJ-45 and nothing else,
with no power and no ground anywhere on it.

The two checks that mattered both hold. The RJ-45 pinout is identical at
both ends, so a straight-through cable is correct -- the pin order runs
opposite between the halves, which is what a part that cannot be mirrored
does, and does not matter since the nets match. And all eighteen keys
keep their exact mesa2 column and row, so one keymap still serves Rev B
and both halves.

Record the review findings as accepted rather than outstanding, and
correct LAYOUT.md: the unconnected GND that DRC reports is a false
positive. The symbol ties the module's ground pads into one net, so DRC
wants copper between them, but the module commons them internally and
the board does not need to.

Assisted-by: Claude:opus-5
Parts:
- removed A1: Pimoroni_Tiny2040, mesa1:Pimoroni_Tiny2040, symbol mesa1:Pimoroni_Tiny2040
- removed C1, C2, C3, C4: 100nF, Capacitor_SMD:C_0603_1608Metric_Pad1.08x0.95mm_HandSolder, symbol Device:C
- removed D1, D_LA1, D_LBK1, D_LE1, D_LI1, D_LN1, D_LO1, D_LS1, D_LSP1, D_LT1: 1N4148W, Diode_SMD:D_SOD-123, symbol Device:D
- removed H1, H3: MountingHole, MountingHole:MountingHole_2.2mm_M2, symbol Mechanical:MountingHole
- removed J2: Tag-Connect TC2030, Connector:Tag-Connect_TC2030-IDC-FP_2x03_P1.27mm_Vertical, symbol Connector_Generic:Conn_02x03_Odd_Even
- removed JP1: SolderJumper_2_Open, Jumper:SolderJumper-2_P1.3mm_Open_RoundedPad1.0x1.5mm, symbol Jumper:SolderJumper_2_Open
- removed LED1, LED2, LED3, LED4: SK6812MINI-HS, mesa1:SK6812-MINI-HS, symbol LED:SK6812
- removed RESET1: RESET_WIRE, TestPoint:TestPoint_Pad_2.0x2.0mm, symbol Connector:TestPoint
- removed SW_LA1, SW_LBK1, SW_LE1, SW_LI1, SW_LN1, SW_LO1, SW_LS1, SW_LSP1, SW_LT1: SW_PG1350, mesa1:Kailh_socket_PG1350, symbol Switch:SW_SPST
- added J1: RJ45, Connector_RJ:RJ45_Amphenol_54602-x08_Horizontal, symbol Connector:RJ45
Connections:
- net COL_1: now also J1.2
- net COL_2: now also J1.3
- net COL_3: now also J1.4
- net COL_4: now also J1.5
- net COL_5: now also J1.8
- net ROW_C: now also J1.7
- net ROW_D: now also J1.6
Other:
- note removed: "Populate diode for voltage drop to led supply. Bypass for full voltage to LEDs"

Commit message: Route both mesa3 halves and finish the right FN key
Rev B is now routed on both hands.  The left half went from bare
placement to 337 segments and 36 vias; the right went from 118 segments
and 7 vias to 149 and 9 as the mode key was wired in.  That key was the
last thing outstanding — on the right the switch and diode were on the
board but deliberately left disconnected, and they now sit at
COL_1/ROW_C, one of the two slots the dropped outer pinky freed,
matching COL_1/ROW_A on the left.  Each half therefore gains one Kailh
socket and one 1N4148W over Rev A.

fnkey.py now places both halves instead of only the left, as its own
docstring said it should when the right-hand key was still undecided.
Each FN key is derived from its own anchor — a local (PITCH, 0) offset
in SW_xE1's frame, carrying that switch's rotation — and the sign flips
on the right, where local +X points outboard rather than inboard.
Because the two halves are computed independently, their mirror
symmetry is a genuine cross-check rather than a restatement of the same
arithmetic, so the script now makes it one: it refuses to write unless
every switch and diode pair sums to 270.0 mm in x, shares a y, and has
opposite rotations.  The hand placement this replaced was 0.846 mm out;
the new keycap clears SW_RE1 by the 0.500 mm target exactly.

apply-fnkey.py follows, walking both boards from a board-keyed
fn-placement.json and saving only the ones that actually moved.  It
still goes through pcbnew rather than Konnect's IPC path, which
continues to segfault KiCAD 10.0.5 on this machine.

Assisted-by: Claude:opus-5
Parts:
- added D_RFN1: 1N4148W, Diode_SMD:D_SOD-123, symbol Device:D
- added SW_RFN1: SW_PG1350, mesa1:Kailh_socket_PG1350, symbol Switch:SW_SPST
Connections:
- net COL_1: now also D_RFN1.1 (K)
- net ROW_C: now also SW_RFN1.1 (A)
- new net: D_RFN1.2 (A), SW_RFN1.2 (B)
Changed lines of the file:
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@@
+	)
+	(junction
+		(at 54.61 83.82)
+		(diameter 0)
+		(color 0 0 0 0)
 	)
 	(junction
@@
 	(wire
 		(pts
-			(xy 54.61 63.5) (xy 54.61 109.22)
+			(xy 54.61 63.5) (xy 54.61 83.82)
 		)
 		(stroke
@@
 	(wire
 		(pts
+			(xy 22.86 83.82) (xy 22.86 74.93)
+		)
+		(stroke
+			(width 0)
+			(type default)
+		)
+	)
+	(wire
+		(pts
 			(xy 25.4 109.22) (xy 22.86 109.22)
 		)
@@
 	(wire
 		(pts
+			(xy 35.56 83.82) (xy 44.45 83.82)
+		)
+		(stroke
+			(width 0)
+			(type default)
+		)
+	)
+	(wire
+		(pts
 			(xy 135.89 85.09) (xy 146.05 85.09)
 		)
@@
 		(pts
 			(xy 73.66 99.06) (xy 73.66 109.22)
+		)
+		(stroke
+			(width 0)
+			(type default)
+		)
+	)
+	(wire
+		(pts
+			(xy 25.4 83.82) (xy 22.86 83.82)
+		)
+		(stroke
+			(width 0)
+			(type default)
+		)
+	)
+	(wire
+		(pts
+			(xy 52.07 83.82) (xy 54.61 83.82)
+		)
+		(stroke
+			(width 0)
+			(type default)
+		)
+	)
+	(wire
+		(pts
+			(xy 54.61 83.82) (xy 54.61 109.22)
 		)
 		(stroke
@@
 	)
 	(symbol
+		(lib_id "Switch:SW_SPST")
+		(at 30.48 83.82 0)
+		(unit 1)
+		(body_style 1)
+		(exclude_from_sim no)
+		(in_bom yes)
+		(on_board yes)
+		(in_pos_files yes)
+		(dnp no)
+		(property "Reference" "SW_RFN1"
+			(at 30.48 80.01 0)
+			(show_name no)
+			(do_not_autoplace no)
+			(effects
+				(font
+					(size 1.27 1.27)
+				)
+			)
+		)
+		(property "Value" "SW_PG1350"
+			(at 30.48 87.63 0)
+			(show_name no)
+			(do_not_autoplace no)
+			(effects
+				(font
+					(size 1.27 1.27)
+				)
+			)
+		)
+		(property "Footprint" "mesa1:Kailh_socket_PG1350"
+			(at 30.48 83.82 0)
+			(hide yes)
+			(show_name no)
+			(do_not_autoplace no)
+			(effects
+				(font
+					(size 1.27 1.27)
+				)
+			)
+		)
+		(property "Datasheet" ""
+			(at 30.48 83.82 0)
+			(hide yes)
+			(show_name no)
+			(do_not_autoplace no)
+			(effects
+				(font
+					(size 1.27 1.27)
+				)
+			)
+		)
+		(property "Description" ""
+			(at 30.48 83.82 0)
+			(show_name no)
+			(do_not_autoplace no)
+			(effects
+				(font
+					(size 1.27 1.27)
+				)
+			)
+		)
+		(pin "2"
+		)
+		(pin "1"
+		)
+		(instances
+			(project "mesa3-right"
+				(path "/6762c7a5-6197-445d-9eb4-2a300e3d331b"
+					(reference "SW_RFN1")
+					(unit 1)
+				)
+			)
+		)
+	)
+	(symbol
 		(lib_id "Mechanical:MountingHole")
 		(at 199.39 152.4 0)
@@
 					(unit 1)
 				)
+			)
+		)
+	)
+	(symbol
+		(lib_id "Device:D")
+		(at 48.26 83.82 180)
+		(unit 1)
+		(body_style 1)
+		(exclude_from_sim no)
+		(in_bom yes)
+		(on_board yes)
+		(in_pos_files yes)
+		(dnp no)
+		(property "Reference" "D_RFN1"
+			(at 48.26 80.01 0)
+			(show_name no)
+			(do_not_autoplace no)
+			(effects
+				(font
+					(size 1.27 1.27)
+				)
+			)
+		)
+		(property "Value" "1N4148W"
+			(at 48.26 87.63 0)
+			(show_name no)
+			(do_not_autoplace no)
+			(effects
+				(font
+					(size 1.27 1.27)
+				)
+			)
+		)
+		(property "Footprint" "Diode_SMD:D_SOD-123"
+			(at 48.26 83.82 0)
+			(hide yes)
+			(show_name no)
+			(do_not_autoplace no)
+			(effects
+				(font
+					(size 1.27 1.27)
+				)
+			)
+		)
+		(property "Datasheet" ""
+			(at 48.26 83.82 0)
+			(hide yes)
+			(show_name no)
+			(do_not_autoplace no)
+			(effects
+				(font
+					(size 1.27 1.27)
+				)
+			)
+		)
+		(property "Description" ""
+			(at 48.26 83.82 0)
+			(show_name no)
+			(do_not_autoplace no)
+			(effects
+				(font
+					(size 1.27 1.27)
+				)
+			)
+		)
+		(pin "2"
+		)
+		(pin "1"
+		)
+		(instances
+			(project "mesa3-right"
+				(path "/6762c7a5-6197-445d-9eb4-2a300e3d331b"
+					(reference "D_RFN1")
+					(unit 1)
+				)
